Commit message: Updated srdf with new update.sh script

File: config/srdf/end_effectors/no-ee.srdf.xacro (robot description, xacro)
@@ -1,5 +1,5 @@
 <?xml version="1.0" ?>
 <robot xmlns:xacro="http://ros.org/wiki/xacro">
-    <xacro:property name="end_effector_name" value="custom" />
+    <xacro:property name="end_effector_name" value="no-ee" />
     <xacro:macro name="define_end_effector" params="arm name">
         <!-- <end_effector name="${name}" parent_link="${arm}_tool_link" group="${name}" parent_group="${arm}_torso" /> -->
